Commit message: urdf finished except for end effector and ros bridge made

File: ROS/urdf/arm.urdf.xacro (robot description, xacro)
@@ -4,5 +4,5 @@
   <xacro:property name="upper_arm_length" value="0.091"/>
   <xacro:property name="forearm_length"   value="0.08"/>
-  <xacro:property name="hand_length"      value="0.033"/>
+  <xacro:property name="hand_length"      value="0.013"/>
   <xacro:property name="upper_arm_diameter" value="0.047"/>
   <xacro:property name="forearm_diameter"   value="0.045"/>
@@ -12,5 +12,6 @@
   <xacro:property name="base_length"        value="0.033"/>
   <xacro:property name="base_diameter"      value="0.09"/>
-  <xacro:property name="shoulder_start_angle" value="30"/>
+  <xacro:property name="shoulder_origin_angle" value="${10+40}"/>
+  <xacro:property name="joint_velocity" value="${pi/2.37}"/>
   <!-- Materials -->
   <material name="blue"><color rgba="0 0 0.8 1"/></material>
@@ -31,7 +32,8 @@
     <parent link="world_link"/>
     <child link="base_link"/>
+    <!--<origin xyz="-.558 0 0" rpy="0 0 0"/>-->
     <origin xyz="0 0 0" rpy="0 0 0"/>
     <axis xyz="0 0 1"/>
-    <limit effort="30" velocity="5" lower="-1.57" upper="1.57"/>
+    <limit effort="30" velocity="5" lower="${20*pi/180}" upper="${170*pi/180}"/>
   </joint>
   <link name="base_link">
@@ -48,7 +50,7 @@
     <parent link="base_link"/>
     <child link="upper_arm"/>
-    <origin xyz="0 0 ${base_length}" rpy="0 -${shoulder_start_angle*pi/180} 0"/>
+    <origin xyz="0 0 ${base_length}" rpy="0 -${shoulder_origin_angle*pi/180} 0"/>
     <axis xyz="0 1 0"/>
-    <limit effort="30" velocity="5" lower="-.4" upper="1.57"/>
+    <limit effort="30" velocity="${joint_velocity}" lower="${40*pi/180}" upper="${80*pi/180}"/>
   </joint>
   <link name="upper_arm">
@@ -70,7 +72,7 @@
     <parent link="upper_arm"/>
     <child link="mid-forearm"/>
-    <origin xyz="0 0 ${upper_arm_length}" rpy="0 ${pi/2} 0"/>
+    <origin xyz="0 0 ${upper_arm_length}" rpy="0 0 0"/>
     <axis xyz="0 1 0"/>
-    <limit effort="30" velocity="5" lower="-1.57" upper="1.57"/>
+    <limit effort="30" velocity="${joint_velocity}" lower="0" upper="${80*pi/180}"/>
   </joint>
  <link name="mid-forearm">
@@ -88,5 +90,5 @@
     <origin xyz="-${midforearm_length} 0 0" rpy="0 0 0"/>
     <axis xyz="1 0 0"/>
-    <limit effort="30" velocity="5" lower="-1.57" upper="1.57"/>
+    <limit effort="30" velocity="${joint_velocity}" lower="-1.57" upper="1.57"/>
   </joint>
   <link name="forearm">
@@ -104,9 +106,9 @@
     <origin xyz="0 0 ${forearm_length}" rpy="0 0 0"/>
     <axis xyz="0 1 0"/>
-    <limit effort="30" velocity="5" lower="-1.57" upper="1.57"/>
+    <limit effort="30" velocity="${joint_velocity}" lower="${60*pi/180}" upper="${120*pi/180}"/>
   </joint>
   <link name="hand">
     <visual>
-      <origin xyz="0 0 ${hand_length/2}" rpy="0 0 0"/>
+      <origin xyz="-.002 0 0" rpy="0 0 0"/>
       <geometry>
         <mesh filename="file:$(arg mesh_path)/End effector.stl" scale=".001 .001 .001"/>
@@ -120,5 +122,5 @@
     <origin xyz="0 0 0" rpy="0 0 0"/>
     <axis xyz="0 1 0"/>
-    <limit effort="30" velocity="5" lower="-.004" upper=".005"/>
+    <limit effort="30" velocity="${joint_velocity}" lower="-.004" upper=".005"/>
   </joint>
   <joint name="hand_to_gripper_left" type="prismatic">
@@ -127,9 +129,9 @@
     <origin xyz="0 0 0" rpy="0 0 0"/>
     <axis xyz="0 1 0"/>
-    <limit effort="30" velocity="5" lower="-.005" upper=".003"/>
+    <limit effort="30" velocity="${joint_velocity}" lower="-.005" upper=".003"/>
   </joint>
   <link name="gripper_right">
     <visual>
-      <origin xyz="-.018 -.01 .017" rpy="0 0 0"/>
+      <origin xyz="-.018 -.01 0" rpy="0 0 0"/>
       <geometry>
         <mesh filename="file:$(arg mesh_path)/Gripper.stl" scale=".001 .001 .001"/>
@@ -140,5 +142,5 @@
   <link name="gripper_left">
     <visual>
-      <origin xyz="-.018 .01 .017" rpy="${pi} 0 0"/>
+      <origin xyz="-.018 .01 0" rpy="${pi} 0 0"/>
       <geometry>
         <mesh filename="file:$(arg mesh_path)/Gripper.stl" scale=".001 .001 .001"/>
