Commit message: Everything except gripper movement works

File: ROS/kinect_arm/urdf/arm.urdf.xacro (robot description, xacro)
@@ -1,151 +1,210 @@
 <?xml version="1.0"?>
 <robot xmlns:xacro="http://ros.org/wiki/xacro" name="kinect_arm">
-  <!-- Properties -->
-  <xacro:property name="upper_arm_length" value="0.091"/>
-  <xacro:property name="forearm_length"   value="0.08"/>
-  <xacro:property name="hand_length"      value="0.013"/>
-  <xacro:property name="upper_arm_diameter" value="0.047"/>
-  <xacro:property name="forearm_diameter"   value="0.045"/>
-  <xacro:property name="midforearm_length"   value="0.035"/>
-  <xacro:property name="hand_diameter"      value="0.0356"/>
-  <xacro:property name="hand_diameter"      value="0.0356"/>
-  <xacro:property name="base_length"        value="0.033"/>
-  <xacro:property name="base_diameter"      value="0.09"/>
-  <xacro:property name="shoulder_origin_angle" value="${10+40}"/>
-  <xacro:property name="joint_velocity" value="${pi/2.37}"/>
-  <!-- Materials -->
-  <material name="blue"><color rgba="0 0 0.8 1"/></material>
-  <material name="red"><color rgba="1 0 0 1"/></material>
-  <material name="yellow"><color rgba="1 1 0 1"/></material>
+    <!-- Properties -->
+    <xacro:property name="upper_arm_length" value="0.091"/>
+    <xacro:property name="forearm_length"   value="0.08"/>
+    <xacro:property name="hand_length"      value="0.013"/>
+    <xacro:property name="upper_arm_diameter" value="0.047"/>
+    <xacro:property name="forearm_diameter"   value="0.045"/>
+    <xacro:property name="midforearm_length"   value="0.035"/>
+    <xacro:property name="hand_diameter"      value="0.0356"/>
+    <xacro:property name="hand_diameter"      value="0.0356"/>
+    <xacro:property name="base_length"        value="0.033"/>
+    <xacro:property name="base_diameter"      value="0.09"/>
+    <xacro:property name="shoulder_origin_angle" value="${10+40}"/>
+    <xacro:property name="joint_velocity" value="${pi/2.37}"/>
+    <!-- Materials -->
+    <material name="blue"><color rgba="0 0 0.8 1"/></material>
+    <material name="red"><color rgba="1 0 0 1"/></material>
+    <material name="yellow"><color rgba="1 1 0 1"/></material>
   <!-- Base Link -->
-  <link name="world_link">
-    <visual>
-      <origin xyz="0 0 0" rpy="0 0 0"/> <!-- Center the geometry -->
-      <geometry>
-        <box size=".001 .001 .001"/>
-      </geometry>
-      <material name="blue"/>
-    </visual>
-  </link>
-  <!-- base_link -> upper_arm -->
-  <joint name="world_to_base" type="revolute">
-    <parent link="world_link"/>
-    <child link="base_link"/>
-    <!--<origin xyz="-.558 0 0" rpy="0 0 0"/>-->
-    <origin xyz="0 0 0" rpy="0 0 0"/>
-    <axis xyz="0 0 1"/>
-    <limit effort="30" velocity="5" lower="${20*pi/180}" upper="${170*pi/180}"/>
-  </joint>
-  <link name="base_link">
-    <visual>
-      <origin xyz="0 0 ${base_length}" rpy="0 0 0"/> <!-- Center the geometry -->
-      <geometry>
-        <!--<cylinder length="${base_length}" radius="${base_diameter/2}"/>-->
-          <mesh filename="file:$(arg mesh_path)/base.stl" scale=".001 .001 .001"/>
-      </geometry>
-      <material name="blue"/>
-    </visual>
-  </link>
-  <joint name="shoulder_joint" type="revolute">
-    <parent link="base_link"/>
-    <child link="upper_arm"/>
-    <origin xyz="0 0 ${base_length}" rpy="0 -${shoulder_origin_angle*pi/180} 0"/>
-    <axis xyz="0 1 0"/>
-    <limit effort="30" velocity="${joint_velocity}" lower="${40*pi/180}" upper="${80*pi/180}"/>
-  </joint>
-  <link name="upper_arm">
-    <visual>
+    <link name="world"/>
+    <!-- base_link -> upper_arm -->
+    <joint name="world_to_base" type="revolute">
+      <parent link="world"/>
+      <child link="base_link"/>
+      <!--<origin xyz="-.558 0 0" rpy="0 0 0"/>-->
       <origin xyz="0 0 0" rpy="0 0 0"/>
-      <geometry>
-          <mesh filename="file:$(arg mesh_path)/upper_arm.stl" scale=".001 .001 .001"/>
-      </geometry>
-      <material name="red"/>
-    </visual>
-    <collision>
-      <origin xyz="0 0 ${upper_arm_length/2}" rpy="0 0 0"/> <!-- Same transform as visual -->
-      <geometry>
-        <cylinder length="${upper_arm_length}" radius="${upper_arm_diameter/2}"/>
-      </geometry>
-  </collision>
-  </link>
-  <joint name="elbow_joint" type="revolute">
-    <parent link="upper_arm"/>
-    <child link="mid-forearm"/>
-    <origin xyz="0 0 ${upper_arm_length}" rpy="0 0 0"/>
-    <axis xyz="0 1 0"/>
-    <limit effort="30" velocity="${joint_velocity}" lower="0" upper="${80*pi/180}"/>
-  </joint>
- <link name="mid-forearm">
-    <visual>
-      <origin xyz="-${midforearm_length/2} 0 0" rpy="0 ${pi/2} 0"/>
-      <geometry>
-        <cylinder length="${midforearm_length}" radius=".0001"/>
-      </geometry>
-      <material name="red"/>
-    </visual>
-  </link>
-  <joint name="sub_elbow_joint" type="fixed">
-    <parent link="mid-forearm"/>
-    <child link="forearm"/>
-    <origin xyz="-${midforearm_length} 0 0" rpy="0 0 0"/>
-    <axis xyz="1 0 0"/>
-    <limit effort="30" velocity="${joint_velocity}" lower="-1.57" upper="1.57"/>
-  </joint>
-  <link name="forearm">
-    <visual>
-      <origin xyz="${midforearm_length} 0 0" rpy="0 0 0"/>
-      <geometry>
-        <mesh filename="file:$(arg mesh_path)/lower_arm.stl" scale=".001 .001 .001"/>
-      </geometry>
-      <material name="red"/>
-    </visual>
-  </link>
-  <joint name="wrist" type="revolute">
-    <parent link="forearm"/>
-    <child link="hand"/>
-    <origin xyz="0 0 ${forearm_length}" rpy="0 0 0"/>
-    <axis xyz="0 1 0"/>
-    <limit effort="30" velocity="${joint_velocity}" lower="${60*pi/180}" upper="${120*pi/180}"/>
-  </joint>
-  <link name="hand">
-    <visual>
-      <origin xyz="-.002 0 0" rpy="0 0 0"/>
-      <geometry>
-        <mesh filename="file:$(arg mesh_path)/End effector.stl" scale=".001 .001 .001"/>
-      </geometry>
-      <material name="yellow"/>
-    </visual>
-  </link>
-  <joint name="hand_to_gripper_right" type="prismatic">
-    <parent link="hand"/>
-    <child link="gripper_right"/>
-    <origin xyz="0 0 0" rpy="0 0 0"/>
-    <axis xyz="0 1 0"/>
-    <limit effort="30" velocity="${joint_velocity}" lower="-.004" upper=".005"/>
-  </joint>
-  <joint name="hand_to_gripper_left" type="prismatic">
-    <parent link="hand"/>
-    <child link="gripper_left"/>
-    <origin xyz="0 0 0" rpy="0 0 0"/>
-    <axis xyz="0 1 0"/>
-    <limit effort="30" velocity="${joint_velocity}" lower="-.005" upper=".003"/>
-  </joint>
-  <link name="gripper_right">
-    <visual>
-      <origin xyz="-.018 -.01 0" rpy="0 0 0"/>
-      <geometry>
-        <mesh filename="file:$(arg mesh_path)/Gripper.stl" scale=".001 .001 .001"/>
-      </geometry>
-      <material name="blue"/>
-    </visual>
-  </link>
-  <link name="gripper_left">
-    <visual>
-      <origin xyz="-.018 .01 0" rpy="${pi} 0 0"/>
-      <geometry>
-        <mesh filename="file:$(arg mesh_path)/Gripper.stl" scale=".001 .001 .001"/>
-      </geometry>
-      <material name="blue"/>
-    </visual>
-  </link>
+      <axis xyz="0 0 1"/>
+      <limit effort="30" velocity="5" lower="${20*pi/180}" upper="${170*pi/180}"/>
+    </joint>
+    <joint name="wrist" type="revolute">
+      <parent link="forearm"/>
+      <child link="hand"/>
+      <origin xyz="0 0 ${forearm_length}" rpy="0 0 0"/>
+      <axis xyz="0 1 0"/>
+      <limit effort="30" velocity="${joint_velocity}" lower="${60*pi/180}" upper="${120*pi/180}"/>
+    </joint>
+    <joint name="shoulder_joint" type="revolute">
+      <parent link="base_link"/>
+      <child link="upper_arm"/>
+      <origin xyz="0 0 ${base_length}" rpy="0 -${shoulder_origin_angle*pi/180} 0"/>
+      <axis xyz="0 1 0"/>
+      <limit effort="30" velocity="${joint_velocity}" lower="${40*pi/180}" upper="${80*pi/180}"/>
+    </joint>
+    <joint name="elbow_joint" type="revolute">
+      <parent link="upper_arm"/>
+      <child link="mid-forearm"/>
+      <origin xyz="0 0 ${upper_arm_length}" rpy="0 0 0"/>
+      <axis xyz="0 1 0"/>
+      <limit effort="30" velocity="${joint_velocity}" lower="0" upper="${80*pi/180}"/>
+    </joint>
+    <joint name="sub_elbow_joint" type="fixed">
+      <parent link="mid-forearm"/>
+      <child link="forearm"/>
+      <origin xyz="-${midforearm_length} 0 0" rpy="0 0 0"/>
+      <axis xyz="1 0 0"/>
+      <limit effort="30" velocity="${joint_velocity}" lower="-1.57" upper="1.57"/>
+    </joint>
+    <joint name="hand_to_gripper_right" type="prismatic">
+      <parent link="hand"/>
+      <child link="gripper_right"/>
+      <origin xyz="0 0 0" rpy="0 0 0"/>
+      <axis xyz="0 1 0"/>
+      <limit effort="30" velocity="${joint_velocity}" lower="-.004" upper=".005"/>
+    </joint>
+    <joint name="hand_to_gripper_left" type="prismatic">
+      <parent link="hand"/>
+      <child link="gripper_left"/>
+      <origin xyz="0 0 0" rpy="0 0 0"/>
+      <axis xyz="0 1 0"/>
+      <limit effort="30" velocity="${joint_velocity}" lower="-.005" upper=".003"/>
+      <mimic joint="hand_to_gripper_right" multiplier="-1.0" offset="0.0"/>
+    </joint>
+    <link name="base_link">
+      <visual>
+        <origin xyz="0 0 ${base_length}" rpy="0 0 0"/> <!-- Center the geometry -->
+        <geometry>
+          <!--<cylinder length="${base_length}" radius="${base_diameter/2}"/>-->
+            <mesh filename="file:$(arg mesh_path)/base.stl" scale=".001 .001 .001"/>
+        </geometry>
+        <material name="blue"/>
+      </visual>
+      <collision>
+        <origin xyz="0 0 ${base_length/2}" rpy="0 0 0"/> <!-- Center the geometry -->
+        <geometry>
+            <cylinder length="${base_length}" radius="${base_diameter/2}"/>
+        </geometry>
+      </collision>
+    </link>
+    <link name="upper_arm">
+      <visual>
+        <origin xyz="0 0 0" rpy="0 0 0"/>
+        <geometry>
+            <mesh filename="file:$(arg mesh_path)/upper_arm.stl" scale=".001 .001 .001"/>
+        </geometry>
+        <material name="red"/>
+      </visual>
+      <collision>
+        <origin xyz="0 0 ${upper_arm_length/2}" rpy="0 0 0"/> <!-- Same transform as visual -->
+        <geometry>
+          <cylinder length="${upper_arm_length}" radius="${upper_arm_diameter/2}"/>
+        </geometry>
+      </collision>
+    </link>
+  <link name="mid-forearm">
+      <visual>
+        <origin xyz="-${midforearm_length/2} 0 0" rpy="0 ${pi/2} 0"/>
+        <geometry>
+          <cylinder length="${midforearm_length}" radius=".0001"/>
+        </geometry>
+        <material name="red"/>
+      </visual>
+      <collision>
+        <origin xyz="-${midforearm_length/2} 0 0" rpy="0 ${pi/2} 0"/>
+        <geometry>
+          <cylinder length="${midforearm_length}" radius=".01"/>
+        </geometry>
+      </collision>
+    </link>
+    <link name="forearm">
+      <visual>
+        <origin xyz="${midforearm_length} 0 0" rpy="0 0 0"/>
+        <geometry>
+          <mesh filename="file:$(arg mesh_path)/lower_arm.stl" scale=".001 .001 .001"/>
+        </geometry>
+        <material name="red"/>
+      </visual>
+      <collision>
+        <origin xyz="0 0 ${forearm_length/2}" rpy="0 0 0"/>
+        <geometry>
+          <cylinder length="${forearm_length}" radius="${forearm_diameter/2}"/>
+        </geometry>
+        <material name="blue"/>
+      </collision>
+    </link>
+    <link name="hand">
+      <visual>
+        <origin xyz="-.002 0 0" rpy="0 0 0"/>
+        <geometry>
+          <mesh filename="file:$(arg mesh_path)/End effector.stl" scale=".001 .001 .001"/>
+        </geometry>
+        <material name="yellow"/>
+      </visual>
+      <collision>
+        <origin xyz="-.002 0 0" rpy="0 0 0"/>
+        <geometry>
+          <cylinder length=".04" radius=".015"/>
+        </geometry>
+        <material name="yellow"/>
+      </collision>
+    </link>
+    <link name="gripper_right">
+      <visual>
+        <origin xyz="-.018 -.01 0" rpy="0 0 0"/>
+        <geometry>
+          <mesh filename="file:$(arg mesh_path)/Gripper.stl" scale=".001 .001 .001"/>
+        </geometry>
+        <material name="blue"/>
+      </visual>
+      <collision>
+        <origin xyz="-.018 -.01 0" rpy="0 0 0"/>
+        <geometry>
+          <box size=".03 .01 .03"/>
+        </geometry>
+        <material name="blue"/>
+      </collision>
+    </link>
+    <link name="gripper_left">
+      <visual>
+        <origin xyz="-.018 .01 0" rpy="${pi} 0 0"/>
+        <geometry>
+          <mesh filename="file:$(arg mesh_path)/Gripper.stl" scale=".001 .001 .001"/>
+        </geometry>
+        <material name="blue"/>
+      </visual>
+      <collision>
+        <origin xyz="-.018 .01 0" rpy="${pi} 0 0"/>
+        <geometry>
+          <box size=".03 .01 .03"/>
+        </geometry>
+        <material name="blue"/>
+      </collision>
+    </link>
+  <ros2_control name="KinectArmHardware" type="system">
+  <hardware>
+    <plugin>mock_components/GenericSystem</plugin>
+  </hardware>
+  <joint name="world_to_base">
+    <command_interface name="position"/>
+    <state_interface name="position"/>
+  </joint>
+  <joint name="shoulder_joint">
+    <command_interface name="position"/>
+    <state_interface name="position"/>
+  </joint>
+  <joint name="elbow_joint">
+    <command_interface name="position"/>
+    <state_interface name="position"/>
+  </joint>
+  <joint name="wrist">
+    <command_interface name="position"/>
+    <state_interface name="position"/>
+  </joint>
+  <joint name="hand_to_gripper_right">
+    <command_interface name="position"/>
+    <state_interface name="position"/>
+    <state_interface name="velocity"/>
+  </joint>
+  </ros2_control>
 </robot>
