Commit message: urdf updated

File: ROS/arm_driver/urdf/arm.urdf.xacro (robot description, xacro)
@@ -5,8 +5,11 @@
     <xacro:property name="forearm_length"   value="0.08"/>
     <xacro:property name="hand_length"      value="0.013"/>
-    <xacro:property name="upper_arm_diameter" value="0.047"/>
-    <xacro:property name="forearm_diameter"   value="0.045"/>
+    <xacro:property name="upper_arm_width" value="0.068"/>
+    <xacro:property name="upper_arm_depth" value="0.038"/>
+    <xacro:property name="forearm_width"   value="0.063"/>
+    <xacro:property name="forearm_depth"   value="0.030"/>
     <xacro:property name="midforearm_length"   value="0.035"/>
-    <xacro:property name="hand_diameter"      value="0.0356"/>
+    <xacro:property name="midforearm_width"   value="${upper_arm_width}"/>
+    <xacro:property name="midforearm_depth"   value="0.035"/>
     <xacro:property name="hand_diameter"      value="0.0356"/>
     <xacro:property name="base_length"        value="0.033"/>
@@ -62,5 +65,5 @@
       <origin xyz="0 0 0" rpy="0 0 0"/>
       <axis xyz="0 1 0"/>
-      <limit effort="30" velocity="${joint_velocity}" lower="-.004" upper=".005"/>
+      <limit effort="30" velocity="${joint_velocity}" lower="-0.005" upper=".002"/>
     </joint>
     <joint name="hand_to_gripper_left" type="prismatic">
@@ -69,5 +72,5 @@
       <origin xyz="0 0 0" rpy="0 0 0"/>
       <axis xyz="0 1 0"/>
-      <limit effort="30" velocity="${joint_velocity}" lower="-.005" upper=".003"/>
+      <limit effort="30" velocity="${joint_velocity}" lower="0" upper=".003"/>
       <mimic joint="hand_to_gripper_right" multiplier="-1.0" offset="0.0"/>
     </joint>
@@ -76,5 +79,4 @@
         <origin xyz="0 0 ${base_length}" rpy="0 0 0"/> <!-- Center the geometry -->
         <geometry>
-          <!--<cylinder length="${base_length}" radius="${base_diameter/2}"/>-->
             <mesh filename="file:$(arg mesh_path)/base.stl" scale=".001 .001 .001"/>
         </geometry>
@@ -99,5 +101,5 @@
         <origin xyz="0 0 ${upper_arm_length/2}" rpy="0 0 0"/> <!-- Same transform as visual -->
         <geometry>
-          <cylinder length="${upper_arm_length}" radius="${upper_arm_diameter/2}"/>
+          <box size="${upper_arm_depth} ${upper_arm_width} ${upper_arm_length}"/>
         </geometry>
       </collision>
@@ -112,7 +114,7 @@
       </visual>
       <collision>
-        <origin xyz="-${midforearm_length/2} 0 0" rpy="0 ${pi/2} 0"/>
-        <geometry>
-          <cylinder length="${midforearm_length}" radius=".01"/>
+        <origin xyz="-${midforearm_length/2 - .002} 0 0" rpy="0 ${pi/2} 0"/>
+        <geometry>
+          <box size="${midforearm_depth} ${midforearm_width} ${midforearm_length + upper_arm_depth/2 + forearm_depth/2}"/>
         </geometry>
       </collision>
@@ -129,5 +131,5 @@
         <origin xyz="0 0 ${forearm_length/2}" rpy="0 0 0"/>
         <geometry>
-          <cylinder length="${forearm_length}" radius="${forearm_diameter/2}"/>
+          <box size="${forearm_depth} ${forearm_width} ${forearm_length}"/>
         </geometry>
         <material name="blue"/>
@@ -143,7 +145,7 @@
       </visual>
       <collision>
-        <origin xyz="-.002 0 0" rpy="0 0 0"/>
-        <geometry>
-          <cylinder length=".04" radius=".015"/>
+        <origin xyz="-.002 0 0" rpy="${pi/2} 0 0"/>
+        <geometry>
+          <cylinder length=".063" radius=".015"/>
         </geometry>
         <material name="yellow"/>

Commit message: simplifying stuff

File: ROS/arm_driver/urdf/arm.urdf.xacro (robot description, xacro)
@@ -44,5 +44,5 @@
       <origin xyz="0 0 ${base_length}" rpy="0 -${shoulder_origin_angle*pi/180} 0"/>
       <axis xyz="0 1 0"/>
-      <limit effort="30" velocity="${joint_velocity}" lower="${40*pi/180}" upper="${80*pi/180}"/>
+      <limit effort="30" velocity="${joint_velocity}" lower="${70*pi/180}" upper="${150*pi/180}"/>
     </joint>
     <joint name="elbow_joint" type="revolute">

Commit message: trying

File: ROS/arm_driver/urdf/arm.urdf.xacro (robot description, xacro)
@@ -15,5 +15,5 @@
     <xacro:property name="base_length"        value="0.033"/>
     <xacro:property name="base_diameter"      value="0.09"/>
-    <xacro:property name="shoulder_origin_angle" value="${10+40}"/>
+    <xacro:property name="shoulder_origin_angle" value="${120}"/>
     <xacro:property name="joint_velocity" value="${pi/2.37}"/>
     <!-- Materials -->

Commit message: thing

File: ROS/arm_driver/urdf/arm.urdf.xacro (robot description, xacro)
@@ -30,5 +30,5 @@
       <origin xyz="0 0 0" rpy="0 0 0"/>
       <axis xyz="0 0 1"/>
-      <limit effort="30" velocity="5" lower="${20*pi/180}" upper="${170*pi/180}"/>
+      <limit effort="30" acceleration="10" velocity="${joint_velocity}" lower="${20*pi/180}" upper="${170*pi/180}"/>
     </joint>
     <joint name="wrist" type="revolute">
@@ -37,5 +37,5 @@
       <origin xyz="0 0 ${forearm_length}" rpy="0 0 0"/>
       <axis xyz="0 1 0"/>
-      <limit effort="30" velocity="${joint_velocity}" lower="${60*pi/180}" upper="${120*pi/180}"/>
+      <limit effort="30" acceleration="10" velocity="${joint_velocity}" lower="${60*pi/180}" upper="${120*pi/180}"/>
     </joint>
     <joint name="shoulder_joint" type="revolute">
@@ -44,5 +44,5 @@
       <origin xyz="0 0 ${base_length}" rpy="0 -${shoulder_origin_angle*pi/180} 0"/>
       <axis xyz="0 1 0"/>
-      <limit effort="30" velocity="${joint_velocity}" lower="${70*pi/180}" upper="${150*pi/180}"/>
+      <limit effort="30" acceleration="10" velocity="${joint_velocity}" lower="${70*pi/180}" upper="${150*pi/180}"/>
     </joint>
     <joint name="elbow_joint" type="revolute">
@@ -51,5 +51,5 @@
       <origin xyz="0 0 ${upper_arm_length}" rpy="0 0 0"/>
       <axis xyz="0 1 0"/>
-      <limit effort="30" velocity="${joint_velocity}" lower="0" upper="${80*pi/180}"/>
+      <limit effort="30" acceleration="10" velocity="${joint_velocity}" lower="0" upper="${80*pi/180}"/>
     </joint>
     <joint name="sub_elbow_joint" type="fixed">
@@ -58,5 +58,5 @@
       <origin xyz="-${midforearm_length} 0 0" rpy="0 0 0"/>
       <axis xyz="1 0 0"/>
-      <limit effort="30" velocity="${joint_velocity}" lower="-1.57" upper="1.57"/>
+      <limit effort="30" acceleration="10" velocity="${joint_velocity}" lower="-1.57" upper="1.57"/>
     </joint>
     <joint name="hand_to_gripper_right" type="prismatic">
@@ -65,5 +65,5 @@
       <origin xyz="0 0 0" rpy="0 0 0"/>
       <axis xyz="0 1 0"/>
-      <limit effort="30" velocity="${joint_velocity}" lower="-0.005" upper=".002"/>
+      <limit effort="30" acceleration="10" velocity="${joint_velocity}" lower="-0.005" upper=".002"/>
     </joint>
     <joint name="hand_to_gripper_left" type="prismatic">
